Commit message: aaaaaaaaaaaa

File: asinus_description/asinus/asinus_2_wheel.urdf.xacro (robot description, xacro)
@@ -3,7 +3,7 @@
   <xacro:arg name="prefix" default="" />
   <xacro:arg name="use_mock_hardware" default="false" />
-  <xacro:include filename="$(find asinus_description)/asinus/robot_4_wheel.urdf" />
+  <xacro:include filename="$(find asinus_description)/asinus/robot_2_wheel.urdf" />
   <!-- Import diffbot ros2_control description -->
-  <xacro:include filename="$(find asinus_description)/asinus/control_4_wheel.xacro" />
+  <xacro:include filename="$(find asinus_description)/asinus/control_2_wheel.xacro" />
   <xacro:asinus_ros2_control
     name="AsinusControl" prefix="$(arg prefix)" use_mock_hardware="$(arg use_mock_hardware)"/>

File: asinus_description/asinus/control_2_wheel.xacro (robot description, xacro)
@@ -5,7 +5,13 @@
       <xacro:unless value="${use_mock_hardware}">
         <hardware>
-          <plugin>asinus_control/DiffBotSystemHardware</plugin>
-          <param name="example_param_hw_start_duration_sec">0</param>
-          <param name="example_param_hw_stop_duration_sec">3.0</param>
+          <plugin>asinus_hardware_interface/AsinusHardwareInterface</plugin>
+          <param name="back_left_wheel_joint_name">${prefix}bl_wheel_joint</param>
+          <param name="back_right_wheel_joint_name">${prefix}br_wheel_joint</param>
+          <param name="loop_rate">50</param>
+          <param name="publish_rate">100</param>
+          <param name="device">/dev/ttyACM1</param>
+          <param name="baud_rate">115200</param>
+          <param name="timeout">1000</param>
+          <param name="encoder_ticks_per_revolution">1024</param>
         </hardware>
       </xacro:unless>
@@ -16,14 +22,4 @@
         </hardware>
       </xacro:if>
-      <joint name="${prefix}fr_wheel_joint">
-        <command_interface name="velocity"/>
-        <state_interface name="position"/>
-        <state_interface name="velocity"/>
-      </joint>
-      <joint name="${prefix}fl_wheel_joint">
-        <command_interface name="velocity"/>
-        <state_interface name="position"/>
-        <state_interface name="velocity"/>
-      </joint>
       <joint name="${prefix}bl_wheel_joint">
         <command_interface name="velocity"/>
