Commit message: Refactor asinus packages and remove unused components
- Updated CMakeLists.txt and package.xml for asinus_nav to remove unnecessary dependencies.
- Deleted asinus_ros2_control package as it was no longer needed.
- Modified asinus_slam package to remove unused RTAB-Map dependencies.
- Added a new Python script (python.py) for converting Twist messages to TwistStamped.
- Removed the ros2_control_asinus package, including its CMakeLists.txt, package.xml, and source files, as it was redundant.
- Cleaned up related launch and configuration files for the removed ros2_control_asinus package.
- Removed associated test files for the deleted ros2_control_asinus package.

File: asinus_description/asinus/control_2_wheel.xacro (robot description, xacro)
@@ -6,12 +6,11 @@
         <hardware>
           <plugin>asinus_hardware_interface/AsinusHardwareInterface</plugin>
-          <param name="back_left_wheel_joint_name">${prefix}bl_wheel_joint</param>
-          <param name="back_right_wheel_joint_name">${prefix}br_wheel_joint</param>
+          <param name="back_left_wheel_joint_name">bl_wheel_joint</param>
+          <param name="back_right_wheel_joint_name">br_wheel_joint</param>
           <param name="loop_rate">50</param>
-          <param name="publish_rate">100</param>
-          <param name="device">/dev/ttyACM1</param>
-          <param name="baud_rate">115200</param>
-          <param name="timeout">1000</param>
-          <param name="encoder_ticks_per_revolution">1024</param>
+          <param name="update_rate">10</param>
+          <param name="encoder_ticks_per_revolution">90</param>
+          <param name="serial_device">/dev/ttyACM1</param>
+          <param name="serial_baud">115200</param>
         </hardware>
       </xacro:unless>
@@ -22,10 +21,10 @@
         </hardware>
       </xacro:if>
-      <joint name="${prefix}bl_wheel_joint">
+      <joint name="bl_wheel_joint">
         <command_interface name="velocity"/>
         <state_interface name="position"/>
         <state_interface name="velocity"/>
       </joint>
-      <joint name="${prefix}br_wheel_joint">
+      <joint name="br_wheel_joint">
         <command_interface name="velocity"/>
         <state_interface name="position"/>

Commit message: update_imu

File: asinus_description/asinus/control_2_wheel.xacro (robot description, xacro)
@@ -6,11 +6,15 @@
         <hardware>
           <plugin>asinus_hardware_interface/AsinusHardwareInterface</plugin>
+          <param name="typeName">asinus_two_wheel</param>
           <param name="back_left_wheel_joint_name">bl_wheel_joint</param>
           <param name="back_right_wheel_joint_name">br_wheel_joint</param>
           <param name="loop_rate">50</param>
           <param name="update_rate">10</param>
-          <param name="encoder_ticks_per_revolution">90</param>
-          <param name="serial_device">/dev/ttyACM1</param>
+          <param name="encoder_ticks_per_revolution">-90</param>
+          <param name="serial_device">/dev/ttyACM0</param>
           <param name="serial_baud">115200</param>
+          <param name="pid_kp">0.4</param>
+          <param name="pid_ki">0.01</param>
+          <param name="pid_kd">0.0</param>
         </hardware>
       </xacro:unless>
@@ -19,4 +23,15 @@
           <plugin>mock_components/GenericSystem</plugin>
           <param name="calculate_dynamics">true</param>
+          <param name="update_rate">50</param>
+          <joint name="bl_wheel_joint">
+            <command_interface name="velocity"/>
+            <state_interface name="position"/>
+            <state_interface name="velocity"/>
+          </joint>
+          <joint name="br_wheel_joint">
+            <command_interface name="velocity"/>
+            <state_interface name="position"/>
+            <state_interface name="velocity"/>
+          </joint>
         </hardware>
       </xacro:if>

File: asinus_description/asinus/robot.urdf (robot description, URDF)
Before this commit: robot asinus_robot, 12 links, 11 joints
Joints:
- joint imu_frame: origin xyz=-0.1575 -0.0534856 0.298 rpy=3.14159 0 0 -> xyz=-0.1575 -0.0534856 0.298 rpy=-1.8735e-16 3.747e-16 -3.14159

File: asinus_description/asinus/robot_4_wheel.urdf (robot description, URDF)
Before this commit: robot asinus_robot, 9 links, 8 joints
Links:
- link depth_cam: mass 1e-9 -> 1e-6
- link imu: mass 1e-9 -> 1e-6
- link lidar: mass 1e-9 -> 1e-6
- link rgb_cam: mass 1e-9 -> 1e-6

File: asinus_gz/urdf/asinus_gz.xacro (robot description, xacro)
@@ -3,7 +3,7 @@
   <xacro:arg name="prefix" default="" />
   <xacro:arg name="use_mock_hardware" default="true" />
-  <!-- Include the assembled robot (which already brings robot.urdf and control.xacro) -->
-  <xacro:include filename="$(find asinus_description)/asinus/asinus.urdf.xacro" />
-  <!-- Gazebo / ros_gz specific bits -->
+  <xacro:include filename="$(find asinus_description)/asinus/robot_2_wheel.urdf" />
+  <!-- Import diffbot ros2_control description -->
+  <xacro:include filename="$(find asinus_description)/asinus/control_2_wheel.xacro" />
   <xacro:include filename="$(find asinus_gz)/urdf/include/gazebo.urdf.xacro" />
 </robot>

File: asinus_gz/urdf/include/gazebo.urdf.xacro (robot description, xacro)
@@ -5,4 +5,6 @@
   <xacro:arg name="namespace" default=""/>
   <xacro:arg name="use_gazebo_ros_control" default="true"/>
+  <!-- Configurable parent link for the Kinect sensor: set to 'kinect_rgb' by default. -->
+  <xacro:arg name="camera_parent" default="kinect_rgb"/>
   <xacro:property name="processed_prefix" value="$(arg frame_prefix_arg)_" />
   <xacro:property name="robot_namespace" value="/$(arg namespace)"/>
@@ -16,20 +18,4 @@
       <plugin>ign_ros2_control/IgnitionSystem</plugin>
     </hardware>
-    <joint name="fl_wheel_joint">
-      <command_interface name="velocity">
-        <param name="min">-3</param>
-        <param name="max">3</param>
-      </command_interface>
-      <state_interface name="position"/>
-      <state_interface name="velocity"/>
-    </joint>
-    <joint name="fr_wheel_joint">
-      <command_interface name="velocity">
-        <param name="min">-3</param>
-        <param name="max">3</param>
-      </command_interface>
-      <state_interface name="position"/>
-      <state_interface name="velocity"/>
-    </joint>
     <joint name="br_wheel_joint">
       <command_interface name="velocity">
@@ -71,5 +57,6 @@
   </xacro:if>
   <!-- Kinect Sensor -->
-  <xacro:sensor_kinect parent="rgb_cam" namespace="$(arg namespace)"/>
+  <!-- Attach Kinect sensor to the configured parent link (default 'kinect_rgb') -->
+  <xacro:sensor_kinect parent="$(arg camera_parent)" namespace="$(arg namespace)"/>
   <!-- GPS Sensor -->
   <xacro:sensor_gps parent="lidar" namespace="$(arg namespace)"/>
